File: tester/board/tester.sch (EAGLE design)
At the start: 25 parts, among them IC1 LM393N

Commit message: Tester schema and board
Parts:
- removed LED1, LED2, LED3: GREEN, led:LED5MM
- removed OK2, OK3, OK4: LTV816, optocoupler:LTV816
- added B1: ARDUINO_UNO_R3_SHIELD_ICSP, SparkFun-Boards:ARDUINO_UNO_R3_SHIELD_ICSP
- added C1: 100uF, SparkFun-Capacitors:100UF-POLAR-RADIAL-2.5MM-25V-20%
- added C2, C3: 100n, rcl:C-EU025-024X044
- added D10, D13, D14, D15, D16, D3, D5, D7, D8: 1N4004, diode:1N4004
- added D2, D4, D6, D9: (no value), SparkFun-LED:LED-FKIT-1206
- added J1, J6, J7, J8: (no value), SparkFun-Connectors:CONN_023.5MM
- added J2, J4: (no value), SparkFun-Connectors:CONN_03-SCREW-5MM
- added J3: POWER_JACK, SparkFun-Connectors:POWER_JACK
- added J5: AVR_SPI_PROG_3X2NS, SparkFun-Connectors:AVR_SPI_PROG_3X2NS
- added K1, K3, K4, K6, K7: G2RA, relay:G2RA
- added PAD1, PAD2, PAD3, PAD4, PAD5, PAD6: WIREPAD1,6/0,9, wirepad:WIREPAD1,6/0,9
- added Q1, Q10, Q2, Q3, Q4, Q5, Q6, Q7, Q8, Q9: 220mA/50V/3.5Ω, SparkFun-DiscreteSemi:MOSFET-NCH-BSS138
- added R17: 100k, rcl:R-EU_R1206
- added R18: 100, rcl:R-EU_R1206
- added R20, R21: 400, rcl:R-EU_R1206
- added R22: 2.74k, rcl:R-EU_R1206
- added R23: 5k, rcl:R-EU_R1206
- added R24, R25, R26: 200, rcl:R-EU_R1206
- added R27: 15k, rcl:R-EU_0204/5
- added R28: 11k, rcl:R-EU_0204/5
- added R29, R30: 100k, rcl:R-EU_0204/5
- added R31: 1k, rcl:R-EU_R1206
- added U$1: APV2111VY, parts:APV2111VY
- added U1: R-78E5.0-1.0, SparkFun-IC-Power:R-78E5.0-1.0
- D1: value 1N4004 -> (none); device diode:1N4004 -> SparkFun-LED:LED-FKIT-1206
- OK1: value LTV816 -> SFH620A; device optocoupler:LTV816 -> optocoupler:SFH620A
- R1, R2: value 200 -> 400; device rcl:R-EU_0204/5 -> rcl:R-EU_R1206
- R10: value 50k -> 882; device rcl:R-EU_0204/5 -> rcl:R-EU_R1206
- R11: value 100k -> 400; device rcl:R-EU_0204/5 -> rcl:R-EU_R1206
- R12: value 200k -> 200; device rcl:R-EU_0204/5 -> rcl:R-EU_R1206
- R13: value 100k -> 246; device rcl:R-EU_0204/5 -> rcl:R-EU_R1206
- R14: value 56k -> 4k; device rcl:R-EU_0204/5 -> rcl:R-EU_R1206
- R15: value 200 -> 1k; device rcl:R-EU_0204/5 -> rcl:R-EU_R1206
- R16: value 100k -> 50k; device rcl:R-EU_0204/5 -> rcl:R-EU_R1206
- R3: device rcl:R-EU_0204/5 -> rcl:R-EU_R1206
- R4: value 5k -> 200k; device rcl:R-EU_0204/5 -> rcl:R-EU_R1206
- R5: value 5k -> 100k; device rcl:R-EU_0204/5 -> rcl:R-EU_R1206
- R6: value 246 -> 56k; device rcl:R-EU_0204/5 -> rcl:R-EU_R1206
- R7: value 882 -> 2.74k; device rcl:R-EU_0204/5 -> rcl:R-EU_R1206
- R8: value 2.74k -> 400; device rcl:R-EU_0204/5 -> rcl:R-EU_R1206
- R9: value 5k -> 200; device rcl:R-EU_0204/5 -> rcl:R-EU_R1206
Connections:
- removed net +12V: R15.2
- removed net N$OPENEVSE_RELAY_1: OK4.C
- removed net N$PILOT: D1.C, OK1.COL, OK2.COL, OK3.COL, R10.2, R12.2
- removed net N$TESTER_A0: IC1A.OUT, R9.2
- removed net N$TESTER_A1: OK4.EMIT, R16.2
- removed net N$TESTER_A2: R12.1, R13.2, R14.1
- removed net N$TESTER_D10: R2.2
- removed net N$TESTER_D13: R1.2
- removed net N$TESTER_D7: R3.2
- removed net OPENEVSE_GND: OK1.C, OK2.C, R6.1, R7.1, R8.1
- new net AC_EARTH: J2.1, K32.S
- new net GFI_15MA: B1.D2, R25.1
- new net GFI_20MA: B1.*D3, R26.1
- new net MISO: B1.MISO, J5.1
- new net MOSI: B1.MOSI, J5.4
- new net N$11: Q1.D, R7.2
- new net N$14: Q4.S, Q6.S, U$1.EM1
- new net N$15: J7.2, PAD2.P
- new net N$17: J4.1, K32.P
- new net N$18: J8.2, PAD5.P, R29.1
- new net N$19: J8.1, PAD6.P, R30.1
- new net N$20: OK1.AC1, R29.2
- new net N$21: OK1.AC2, R30.2
- new net N$22: C3.1, J3.PWR, U1.IN
- new net N$23: D15.A, K61.2, Q9.D
- new net N$24: D4.A, R8.2
- new net N$25: D16.A, K71.2, Q10.D
- new net N$26: K72.P, R28.2
- new net N$27: Q8.G, R21.2
- new net N$28: K62.P, R27.2
- new net N$29: PAD4.P, R27.1, R28.1
- new net N$30: D14.A, K41.2, Q8.D
- new net N$31: Q2.D, R10.2
- new net N$32: D10.A, K11.2, Q5.D
- new net N$33: Q5.G, R20.2
- new net N$34: D5.C, R10.1
- new net N$35: Q9.G, R25.2
- new net N$36: Q10.G, R26.2
- new net N$37: D1.A, R1.2
- new net N$38: D9.A, R18.2, U$1.A1
- new net N$39: Q7.G, R24.2
- new net N$40: D13.A, K31.2, Q7.D
- new net N$43: Q4.G, Q6.G, U$1.CL1
- new net OPEN_EVSE_AC_H: J4.3, K12.P
- new net OPEN_EVSE_AC_TEST: B1.D13, R21.1
- new net OPEN_EVSE_AC_TEST_H: J6.2, K42.P
- new net OPEN_EVSE_GND: B1.*D11, R24.1
- new net OPEN_EVSE_PILOT: D3.A, D5.A, D7.A, D8.A, J1.2, R22.1, R4.1
- new net OPEN_EVSE_PWR: B1.D12, R20.1
- new net PILOT_VOLTAGE: B1.A0, R4.2, R5.1, R6.2
- new net PWM_READ: B1.*D10, IC1A.OUT, R23.2
- new net RELAY_READ: B1.D4, OK1.C, R31.1
- new net RESET: B1.!RESET!@2, J5.5
- new net SCK: B1.SCK, J5.3
- new net STATE_A: B1.*D5, R1.1
- new net STATE_B: B1.*D6, R2.1, R3.1
- new net STATE_C: B1.D7, R8.1, R9.1
- new net STATE_D: B1.D8, R11.1, R12.1
- new net STATE_E: B1.*D9, R18.1
- new net V_AC_H: J2.3, K12.S, K42.S, K62.S, K72.S
- new net V_AC_L: J2.2, J4.2, J6.1, PAD1.P
- net +5V: now also B1.5V, B1.VCC, C1.+, C2.1, D10.C, D13.C, D14.C, D15.C, D16.C, IC1P.V+, J5.2, K11.1, K31.1, K41.1, K61.1, K71.1, R14.1, R23.1, R31.2, R6.1, U1.OUT; no longer OK4.COL, R14.2, R4.2
- net GND: now also B1.GND, B1.GND@0, B1.GND@1, B1.GND@2, C1.-, C2.2, C3.2, D1.C, D2.C, D4.C, D6.C, D9.C, IC1P.V-, J1.1, J3.GND, J3.GNDBREAK, J5.6, OK1.E, Q1.S, Q10.S, Q2.S, Q3.S, Q5.S, Q6.D, Q7.S, Q8.S, Q9.S, R15.2, R17.2, R5.2, U$1.C1, U1.GND; no longer OK3.C, R11.1, R13.1, R16.1, R5.1, R9.1
- net N$1: now also Q1.G, R3.2; no longer OK1.EMIT, R8.2
- net N$10: now also R14.2, R15.1; no longer R4.1, R5.2
- net N$12: now also R16.2, R17.1; no longer R10.1, R11.2
- net N$13: now also D8.C, R16.1; no longer D1.A
- net N$16: now also Q4.D, R22.2; no longer OK4.A, R15.1
- net N$2: now also D2.A, R2.2; no longer LED1.C, OK1.A
- net N$3: now also D3.C, R7.1; no longer LED1.A, R1.1
- net N$4: now also Q2.G, R9.2; no longer LED2.C, OK2.A
- net N$5: now also D6.A, R11.2; no longer LED2.A, R2.1
- net N$6: now also Q3.G, R12.2; no longer LED3.C, OK3.A
- net N$7: now also D7.C, R13.1; no longer LED3.A, R3.1
- net N$8: now also Q3.D, R13.2; no longer OK2.EMIT, R7.2
- net N$9: now also J7.1, PAD3.P; no longer OK3.EMIT, R6.2
Other:
- note removed: "EV states"
- note removed: "OPENEVSE + 12V"
- note removed: "PWM measurement"
- note removed: "Pilot voltage"
- note removed: "Read relay state"
- moved on the sheet: R1, R10, R11, R12, R13, R14, R15, R16, R2, R3, R4, R5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
